File: KiCAD/PCB/Slab40_PCB.kicad_pcb (KiCad board)
At the start: 2 copper layers, 248 x 85.8 mm, 87 parts, among them SW1 SW_Push, SW10 SW_Push, SW11 SW_Push, SW12 SW_Push, SW13 SW_Push, SW14 SW_Push, SW15 SW_Push, SW16 SW_Push, SW17 SW_Push, SW18 SW_Push, SW19 SW_Push, SW2 SW_Push, SW20 SW_Push, SW21 SW_Push, SW22 SW_Push, SW23 SW_Push, SW24 SW_Push, SW25 SW_Push, SW26 SW_Push, SW27 SW_Push, SW28 SW_Push, SW29 SW_Push, SW3 SW_Push, SW30 SW_Push, SW31 SW_Push, SW32 SW_Push, SW33 SW_Push, SW34 SW_Push, SW35 SW_Push, SW36 SW_Push, SW37 SW_Push, SW38 SW_Push, SW39 SW_Push, SW4 SW_Push, SW40 SW_Push, SW41 SW_Push, SW5 SW_Push, SW6 SW_Push, SW7 SW_Push, SW8 SW_Push, SW9 SW_Push, U1 rp2040-tiny

Commit message: マージンを左右対称に調整
Other:
- board size 248 x 85.8 mm -> 247.6 x 85.8 mm
Changed lines of the file:
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@@
   (title_block
     (title "Slab40 PCB")
-    (date "2024-08-09")
+    (date "2024-09-04")
     (rev "v1.0")
     (company "@ymkn")
@@
     )
   )
-  (gr_line (start 341.25 128.625) (end 97.25 128.625)
+  (gr_line (start 340.9 128.625) (end 97.25 128.625)
     (stroke (width 0.1) (type default)) (layer "Edge.Cuts"))
   (gr_arc (start 97.25 128.625) (mid 95.835786 128.039214) (end 95.25 126.625)
     (stroke (width 0.1) (type default)) (layer "Edge.Cuts"))
-  (gr_line (start 343.25 44.825) (end 343.25 126.625)
+  (gr_line (start 342.9 44.825) (end 342.9 126.625)
     (stroke (width 0.1) (type default)) (layer "Edge.Cuts"))
   (gr_arc (start 95.25 44.825) (mid 95.835786 43.410786) (end 97.25 42.825)
     (stroke (width 0.1) (type default)) (layer "Edge.Cuts"))
-  (gr_line (start 97.25 42.825) (end 341.25 42.825)
+  (gr_line (start 97.25 42.825) (end 340.9 42.825)
     (stroke (width 0.1) (type default)) (layer "Edge.Cuts"))
   (gr_line (start 95.25 126.625) (end 95.25 44.825)
     (stroke (width 0.1) (type default)) (layer "Edge.Cuts"))
-  (gr_arc (start 343.25 126.625) (mid 342.664214 128.039214) (end 341.25 128.625)
+  (gr_arc (start 342.9 126.625) (mid 342.314214 128.039214) (end 340.9 128.625)
     (stroke (width 0.1) (type default)) (layer "Edge.Cuts"))
-  (gr_arc (start 341.25 42.825) (mid 342.664214 43.410786) (end 343.25 44.825)
+  (gr_arc (start 340.9 42.825) (mid 342.314214 43.410786) (end 342.9 44.825)
     (stroke (width 0.1) (type default)) (layer "Edge.Cuts"))
   (gr_text "Slab40 v1.0 by @ymkn" (at 99.05 126.525) (layer "F.SilkS")
@@
   )
   (dimension (type aligned) (layer "Cmts.User")
-    (pts (xy 95.25 47.625) (xy 343.25 47.625))
+    (pts (xy 95.25 47.625) (xy 342.9 47.625))
     (height -6.9)
-    (gr_text "248.0000 mm" (at 219.25 38.575) (layer "Cmts.User")
+    (gr_text "247.6500 mm" (at 219.075 38.575) (layer "Cmts.User")
       (effects (font (size 2 2) (thickness 0.15)))
     )
@@
   )
   (dimension (type aligned) (layer "Cmts.User")
-    (pts (xy 95.25 42.825) (xy 95.25 128.625))
+    (pts (xy 97.75 42.825) (xy 97.75 128.625))
     (height 9.6)
-    (gr_text "85.8000 mm" (at 83.5 85.725 90) (layer "Cmts.User")
+    (gr_text "85.8000 mm" (at 86 85.725 90) (layer "Cmts.User")
       (effects (font (size 2 2) (thickness 0.15)))
     )
