File: KiCAD/SwitchPlate/Slab40_SwitchPlate.kicad_pcb (KiCad board)
At the start: 2 copper layers, 264.1 x 96.8 mm, 45 parts, among them SW1 SW_Push, SW10 SW_Push, SW11 SW_Push, SW12 SW_Push, SW13 SW_Push, SW14 SW_Push, SW15 SW_Push, SW16 SW_Push, SW17 SW_Push, SW18 SW_Push, SW19 SW_Push, SW2 SW_Push, SW20 SW_Push, SW21 SW_Push, SW22 SW_Push, SW23 SW_Push, SW24 SW_Push, SW25 SW_Push, SW26 SW_Push, SW27 SW_Push, SW28 SW_Push, SW29 SW_Push, SW3 SW_Push, SW30 SW_Push, SW31 SW_Push, SW32 SW_Push, SW33 SW_Push, SW34 SW_Push, SW35 SW_Push, SW37 SW_Push, SW38 SW_Push, SW39 SW_Push, SW4 SW_Push, SW40 SW_Push, SW41 SW_Push, SW5 SW_Push, SW6 SW_Push, SW7 SW_Push, SW8 SW_Push, SW9 SW_Push

Commit message: マージンを左右対称に調整
Parts:
- moved REF** 0.22 mm to (90.6, 40.9)
- moved REF** 0.22 mm to (90.6, 130.5)
- moved REF** 0.22 mm to (347.4, 130.5)
- moved REF** 0.22 mm to (347.4, 40.9)
Changed lines of the file:
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@@
   (title_block
     (title "Slab40 SwitchPlate")
-    (date "2024-08-09")
+    (date "2024-09-04")
     (rev "v1.0")
     (company "@ymkn")
@@
   (net 0 "")
   (footprint "MountingHole:MountingHole_3.2mm_M3" (layer "F.Cu")
-    (at 347.65 130.525)
+    (at 347.425 130.525)
     (descr "Mounting Hole 3.2mm, no annular, M3")
     (tags "mounting hole 3.2mm no annular m3")
@@
   )
   (footprint "MountingHole:MountingHole_3.2mm_M3" (layer "F.Cu")
-    (at 347.65 40.925)
+    (at 347.425 40.925)
     (descr "Mounting Hole 3.2mm, no annular, M3")
     (tags "mounting hole 3.2mm no annular m3")
@@
   )
   (footprint "MountingHole:MountingHole_3.2mm_M3" (layer "F.Cu")
-    (at 90.85 40.925)
+    (at 90.625 40.925)
     (descr "Mounting Hole 3.2mm, no annular, M3")
     (tags "mounting hole 3.2mm no annular m3")
@@
   )
   (footprint "MountingHole:MountingHole_3.2mm_M3" (layer "F.Cu")
-    (at 90.85 130.525)
+    (at 90.625 130.525)
     (descr "Mounting Hole 3.2mm, no annular, M3")
     (tags "mounting hole 3.2mm no annular m3")
@@
       (stroke (width 0.05) (type solid)) (layer "Edge.Cuts"))
   )
-  (gr_rect (start 361.85 25.625) (end 381.05 40.625)
-    (stroke (width 0.15) (type default)) (fill none) (layer "B.SilkS"))
-  (gr_line (start 347.35 134.125) (end 91.25 134.125)
+  (gr_line (start 347.125 134.125) (end 91.025 134.125)
     (stroke (width 0.1) (type default)) (layer "Edge.Cuts"))
-  (gr_line (start 351.35 41.325) (end 351.35 130.125)
+  (gr_line (start 351.125 41.325) (end 351.125 130.125)
     (stroke (width 0.1) (type default)) (layer "Edge.Cuts"))
-  (gr_line (start 91.25 37.325) (end 347.35 37.325)
+  (gr_line (start 91.025 37.325) (end 347.125 37.325)
     (stroke (width 0.1) (type default)) (layer "Edge.Cuts"))
-  (gr_arc (start 351.35 130.125) (mid 350.178427 132.953427) (end 347.35 134.125)
+  (gr_arc (start 351.125 130.125) (mid 349.953427 132.953427) (end 347.125 134.125)
     (stroke (width 0.1) (type default)) (layer "Edge.Cuts"))
-  (gr_line (start 87.25 130.125) (end 87.25 41.325)
+  (gr_line (start 87.025 130.125) (end 87.025 41.325)
     (stroke (width 0.1) (type default)) (layer "Edge.Cuts"))
-  (gr_arc (start 87.25 41.325) (mid 88.421573 38.496573) (end 91.25 37.325)
+  (gr_arc (start 87.025 41.325) (mid 88.196573 38.496573) (end 91.025 37.325)
     (stroke (width 0.1) (type default)) (layer "Edge.Cuts"))
-  (gr_arc (start 91.25 134.125) (mid 88.421573 132.953427) (end 87.25 130.125)
+  (gr_arc (start 91.025 134.125) (mid 88.196573 132.953427) (end 87.025 130.125)
     (stroke (width 0.1) (type default)) (layer "Edge.Cuts"))
-  (gr_arc (start 347.35 37.325) (mid 350.178427 38.496573) (end 351.35 41.325)
+  (gr_arc (start 347.125 37.325) (mid 349.953427 38.496573) (end 351.125 41.325)
     (stroke (width 0.1) (type default)) (layer "Edge.Cuts"))
   (gr_text "Slab40 v1.0 by @ymkn" (at 342.35 130.925) (layer "B.SilkS")
@@
   )
   (dimension (type aligned) (layer "Cmts.User")
-    (pts (xy 87.25 41.325) (xy 351.35 41.325))
+    (pts (xy 87.05 41.325) (xy 351.15 41.325))
     (height -12.9)
-    (gr_text "264.1000 mm" (at 219.3 26.275) (layer "Cmts.User")
+    (gr_text "264.1000 mm" (at 219.1 26.275) (layer "Cmts.User")
       (effects (font (size 2 2) (thickness 0.15)))
     )
     (format (prefix "") (suffix "") (units 3) (units_format 1) (precision 4))
+    (style (thickness 0.15) (arrow_length 1.27) (text_position_mode 0) (extension_height 0.58642) (extension_offset 0.5) keep_text_aligned)
+  )
+  (dimension (type aligned) (layer "Cmts.User")
+    (pts (xy 342.9 123.825) (xy 351.125 123.825))
+    (height 15.6)
+    (gr_text "8.2250 mm" (at 347.0125 138.275) (layer "Cmts.User")
+      (effects (font (size 1 1) (thickness 0.15)))
+    )
+    (format (prefix "") (suffix "") (units 3) (units_format 1) (precision 4))
+    (style (thickness 0.15) (arrow_length 1.27) (text_position_mode 0) (extension_height 0.58642) (extension_offset 0.5) keep_text_aligned)
+  )
+  (dimension (type aligned) (layer "Cmts.User")
+    (pts (xy 342.9 123.825) (xy 342.9 134.125))
+    (height -13.325)
+    (gr_text "10.3000 mm" (at 355.075 128.975 90) (layer "Cmts.User")
+      (effects (font (size 1 1) (thickness 0.15)))
+    )
+    (format (prefix "") (suffix "") (units 3) (units_format 1) (precision 4))
+    (style (thickness 0.15) (arrow_length 1.27) (text_position_mode 0) (extension_height 0.58642) (extension_offset 0.5) keep_text_aligned)
+  )
+  (dimension (type aligned) (layer "Cmts.User")
+    (pts (xy 95.25 47.625) (xy 95.25 37.325))
+    (height -15)
+    (gr_text "10.3000 mm" (at 79.1 42.475 90) (layer "Cmts.User")
+      (effects (font (size 1 1) (thickness 0.15)))
+    )
+    (format (prefix "") (suffix "") (units 3) (units_format 1) (precision 4))
+    (style (thickness 0.15) (arrow_length 1.27) (text_position_mode 0) (extension_height 0.58642) (extension_offset 0.5) keep_text_aligned)
+  )
+  (dimension (type aligned) (layer "Cmts.User")
+    (pts (xy 95.25 47.625) (xy 87.025 47.625))
+    (height 13.925)
+    (gr_text "8.2250 mm" (at 91.1375 32.55) (layer "Cmts.User")
+      (effects (font (size 1 1) (thickness 0.15)))
+    )
+    (format (prefix "") (suffix "") (units 3) (units_format 1) (precision 4))
